File: regulator.sch (EAGLE design)
At the start: 26 parts, among them K1 RELAY-SPDT, K2 RELAY-SPDT, T1 BC337, U1 LM393N, U2 TL431PTH

Commit message: Completed the schematics
Parts:
- added R11: 10k, rcl:R-EU_0204/7
- added R12: 4.2k, rcl:R-EU_0204/7
- R3: value 10k -> 47
- R4: value 220 -> 10k
- R5: value 22k -> 100
- R6: value 47k -> 4.7k
- R7: value 4.2k -> 4.7k
- R8: value 4.7k -> 220
- R9: value 4.7k -> 100k
Connections:
- removed net N$4: D4.C
- removed net VDB_B12: R5.1, R6.2, U1.NEG_B
- removed net VDB_B14: R1.2, R2.1
- new net N$3: R11.2, T1.E
- new net VDB: R1.2, R2.1, U1.NEG_B, U1.POA_A
- new net VDD: R3.2, R4.1, R5.2, U1.POS_B
- net +12V: now also D4.C, R12.2, R6.2; no longer D4.A, R8.2, R9.2
- net B+: no longer R5.2
- net COLL: now also D4.A
- net D+: now also R4.2; no longer U1.POS_B
- net GND: now also R11.1, R3.1, R9.2; no longer R3.2, R6.1, T1.E
- net N$1: now also R8.2, R9.1; no longer R3.1, R4.2
- net S_A: now also R6.1; no longer R4.1
- net S_B: now also R5.1, R7.1; no longer R9.1
- net VREF: now also R12.1; no longer R7.1, U1.POA_A
Other:
- note added: "Regulating outputs"
- moved on the sheet: D4, R1, R2, R3, R4, R5, R6, R7, R8, R9
